File: ecad/dbz-radar/dbz-radar.kicad_sch (KiCad schematic)
At the start: 24 parts, among them J1 USB_C_Receptacle_USB2.0_14P, U1 ESP32-S3-WROOM-1, U2 USBLC6-2SC6, U3 AP2112K-3.3

Commit message: copy Qualia design
Parts:
- added C10, C13, C14, C15: 100nF, symbol Device:C_Small
- added C11, C12, C8: 1uF, symbol Device:C_Small
- added C9: 10uF, symbol Device:C_Small
- added D4: MBR0540, Diode_SMD:D_SOD-123, symbol Diode:MBR0540
- added J2: Conn_01x40, symbol Connector_Generic:Conn_01x40
- added L1: L_Small, symbol Device:L_Small
- added R10: 8.2, symbol Device:R_Small_US
- added R11, R12, R14, R21, R22, R23, R25, R27, R32: 0, symbol Device:R_Small_US
- added R13, R15, R24, R26, R28, R29, R30, R31: DNI, symbol Device:R_Small_US
- added R16, R18, R19, R20, R8, R9: 5.1k, symbol Device:R_Small_US
- added R17: 100, symbol Device:R_Small_US
- added SW1, SW2: SW_Push, symbol Switch:SW_Push
- added TP10, TP11, TP12, TP13, TP14, TP15, TP4, TP5, TP6, TP7, TP8, TP9: TestPoint, symbol Connector:TestPoint
- added U4: TPS61169, symbol TPS61169:TPS61169
- added U5, U6: PCA9554, symbol PCA9554:PCA9554
Connections:
- net +3V3: now also C14.1, C15.1, J2.39 (Pin_39), J2.5 (Pin_5), R12.2, R14.2, R16.2, R18.2, R19.2, R20.2, R21.1, R22.1, R23.1, R25.1, R27.1, R30.1, R8.1, R9.1, SW1.2, U5.16 (VCC), U6.16 (VCC)
- net +5V: now also C10.1, C9.1, L1.1, U4.5 (VIN)
- net GND: now also C10.2, C11.1, C12.1, C13.2, C14.2, C15.2, C8.1, C9.2, J2.34 (Pin_34), J2.4 (Pin_4), J2.40 (Pin_40), R10.2, R13.1, R15.1, R24.2, R26.2, R28.1, R29.1, R31.2, R32.2, SW1.1, SW2.1, U4.2 (GND), U5.8 (GND), U6.8 (GND)
- net USB_D+: now also U1.14 (USB_D+)
- net USB_D-: now also U1.13 (USB_D-)
- net A0: now reaches U1.10 (IO17)
- net A0: now also TP11.1
- net SCL: now reaches U1.11 (IO18)
- net SCL: now also J2.37 (Pin_37), R20.1, U5.14 (SCL), U6.14 (SCL)
- net SDA: now reaches U1.12 (IO8)
- net SDA: now also J2.36 (Pin_36), R18.1, U5.15 (SDA), U6.15 (SDA)
- net R5: now reaches U1.15 (IO3)
- net R5: now also J2.33 (Pin_33)
- net R4: now reaches U1.16 (IO46)
- net R4: now also J2.32 (Pin_32)
- net R3: now reaches U1.17 (IO9)
- net R3: now also J2.31 (Pin_31)
- net R2: now reaches U1.18 (IO10)
- net R2: now also J2.30 (Pin_30)
- net R1: now reaches U1.19 (IO11)
- net R1: now also J2.28 (Pin_28), J2.29 (Pin_29)
- net G5: now reaches U1.20 (IO12)
- net G5: now also J2.27 (Pin_27)
- net G4: now reaches U1.21 (IO13)
- net G4: now also J2.26 (Pin_26)
- net G3: now reaches U1.22 (IO14)
- net G3: now also J2.25 (Pin_25)
- net G2: now reaches U1.23 (IO21)
- net G2: now also J2.24 (Pin_24)
- net at U1.24 (IO47): no longer names the net of U1.24 (IO47)
- net at U1.24 (IO47): now also U1.31 (IO38), J2.19 (Pin_19), J2.23 (Pin_23)
- net G0: now reaches U1.25 (IO48)
- net G0: now also J2.22 (Pin_22)
- net B5: now reaches U1.26 (IO45)
- net B5: now also J2.21 (Pin_21)
- net BOOT0_B4: now reaches U1.27 (IO0)
- net BOOT0_B4: now also J2.20 (Pin_20), SW2.2
- net at U1.28 (IO35): now also TP7.1
- net at U1.29 (IO36): now also TP8.1
- net ~{RESET}: now reaches U1.3 (EN)
- net ~{RESET}: now also C8.2, R8.2, TP4.1
- net at U1.30 (IO37): now also TP9.1
- net B2: now reaches U1.32 (IO39)
- net B2: now also J2.18 (Pin_18)
- net B1: now reaches U1.33 (IO40)
- net B1: now also J2.16 (Pin_16), J2.17 (Pin_17)
- net HSYNC: now reaches U1.34 (IO41)
- net HSYNC: now also J2.15 (Pin_15)
- net VSYNC: now reaches U1.35 (IO42)
- net VSYNC: now also J2.14 (Pin_14)
- net RXD0: now reaches U1.36 (RXD0)
- net TXD0: now reaches U1.37 (TXD0)
- net DE: now reaches U1.38 (IO2)
- net DE: now also J2.13 (Pin_13)
- net PCLK: now reaches U1.39 (IO1)
- net at U1.4 (IO4): now also TP10.1
- net SCK: now reaches U1.5 (IO5)
- net MISO: now reaches U1.6 (IO6)
- net MOSI: now reaches U1.7 (IO7)
- net CS: now reaches U1.8 (IO15)
- net CS: now also R19.1
- net A1: now reaches U1.9 (IO16)
- net A1: now also R11.1, TP12.1
- new net: R30.2, R32.1, U6.1 (A0)
- new net: R21.2, R31.1, U6.2 (A1)
- new net: R22.2, R29.2, U6.3 (A2)
- new net: TP14.1, U5.10 (P5)
- new net: R11.2, R9.2, TP13.1, U4.4 (CTRL)
- new net: D4.2 (A), L1.2, U4.1 (SW)
- new net: R25.2, R26.1, U5.2 (A1)
- new net: R23.2, R24.1, U5.1 (A0)
- new net: TP15.1, U5.11 (P6)
- new net: R27.2, R28.2, U5.3 (A2)
- new net +24V: C11.2, C12.2, D4.1 (K), J2.1 (Pin_1), TP5.1
- new net BACKLIGHT: U5.9 (P4)
- new net EXP_IRQ: U5.13 (~{INT})
- new net IM0: J2.8 (Pin_8), R14.1, R15.2
- new net IM1: J2.7 (Pin_7), R12.1, R13.2
- new net LEDK: C13.1, J2.2 (Pin_2), J2.3 (Pin_3), R10.1, TP6.1, U4.3 (FB)
- new net PCLK_CONN: J2.12 (Pin_12), R17.2
- new net PLCK: R17.1
- new net TFT_CS: J2.11 (Pin_11), R16.1, U5.5 (P1)
- new net TFT_MOSI: J2.9 (Pin_9), U5.12 (P7)
- new net TFT_RESET: J2.38 (Pin_38), J2.6 (Pin_6), U5.6 (P2)
- new net TFT_SCK: J2.10 (Pin_10), U5.4 (P0)
- new net TP_IRQ: J2.35 (Pin_35), U5.7 (P3)
- no-connect marks 3 -> 0
Other:
- moved on the sheet: C7, U1

Commit message: add battery charging, monitoring, display, and SD card
Parts:
- removed C15: 100nF, symbol Device:C_Small
- removed R21, R22, R32: 0, symbol Device:R_Small_US
- removed R29, R30, R31: DNI, symbol Device:R_Small_US
- removed TP10, TP11, TP14, TP15, TP7, TP8, TP9: TestPoint, symbol Connector:TestPoint
- removed U6: PCA9554, symbol PCA9554:PCA9554
- added C16, C18: 10uF, symbol Device:C_Small
- added C17, C20, C21: 100nF, symbol Device:C_Small
- added C19: 1uF, symbol Device:C_Small
- added D10, D11, D12, D13, D7, D8, D9: ESD5Zxx, Diode_SMD:D_SOD-523, symbol Diode:ESD5Zxx
- added D14, D6: LED_Small, symbol Device:LED_Small
- added D5: MBR0540, Diode_SMD:D_SOD-123, symbol Diode:MBR0540
- added J3: JST-PH, symbol Connector_Generic_MountingPin:Conn_01x02_MountingPin
- added Q1: Q_PMOS, symbol Device:Q_PMOS
- added R33, R36, R67, R68, R69, R70, R71, R72: 5.1k, symbol Device:R_Small_US
- added R34, R35, R38, R39, R40, R41, R42, R43, R44, R45, R46, R47, R48, R49, R50, R51, R52, R53, R54, R55, R56, R57, R58, R59, R60, R61, R62, R63, R64, R65, R66: 0, symbol Device:R_Small_US
- added R37, R73: 100, symbol Device:R_Small_US
- added TP11, TP14, TP15, TP18, TP19, TP20, TP21, TP22, TP23, TP7, TP8, TP9: TestPoint_Alt, symbol Connector:TestPoint_Alt
- added TP16, TP17: TestPoint, symbol Connector:TestPoint
- added U7: MCP738311/2, symbol MCP7383X:MCP7383X
- added U8: MAX17048/9, symbol MAX17048-9:MAX17048/9
- added U9: 5033981892, symbol 5033981892:5033981892
Connections:
- net +3V3: now also C10.1, C6.2, C9.1, L1.1, R12.1, U4.5 (VIN), C19.1, C20.1, C21.1, D11.1 (K), R68.2, R69.2, R70.2, R71.2, R72.2, U8.3 (Vdd), U9.4 (VDD); no longer C6.1, R12.2
- net B1: now also R60.2; no longer U1.33 (IO40)
- net B2: now also R59.2; no longer U1.32 (IO39)
- net B5: now also R63.2; no longer U1.26 (IO45)
- net BOOT0_B4: now also R40.1; no longer U1.27 (IO0)
- net DE: now also R42.1; no longer U1.38 (IO2)
- net G0: now also R66.2; no longer U1.25 (IO48)
- net G2: now also R57.2; no longer U1.23 (IO21)
- net G3: now also R54.1; no longer U1.22 (IO14)
- net G4: now also R53.1; no longer U1.21 (IO13)
- net G5: now also R52.1; no longer U1.20 (IO12)
- net GND: now also C6.1, R15.2, C16.1, C17.1, C18.2, C19.2, C20.2, C21.2, D10.2 (A), D11.2 (A), D12.2 (A), D13.2 (A), D7.2 (A), D8.2 (A), D9.2 (A), J3.1 (Pin_1), J3.MP (MountPin), R33.1, R36.2, R67.1, R73.1, U7.2 (Vss), U8.1 (CTG), U8.4 (GND), U8.EP, U9.11 (MP0), U9.12 (MP1), U9.13 (MP2), U9.14 (MP3), U9.6 (VSS); no longer C6.2, R15.1
- net HSYNC: now also R61.2; no longer U1.34 (IO41)
- net IM0: now also R12.2, R13.2; no longer R14.1, R15.2
- net IM1: now also R14.1, R15.1; no longer R12.1, R13.2
- net MISO: now also D13.1 (K), R46.1, R71.1, U9.7 (DAT0); no longer U1.6 (IO6)
- net MOSI: now also D10.1 (K), R47.1, R70.1, U9.3 (CMD); no longer U1.7 (IO7)
- net PCLK: now also R41.1; no longer U1.39 (IO1)
- net R1: now also R51.1; no longer U1.19 (IO11)
- net R2: now also R50.1; no longer U1.18 (IO10)
- net R3: now also R49.1; no longer U1.17 (IO9)
- net R4: now also R64.2; no longer U1.16 (IO46)
- net R5: now also R43.1; no longer U1.15 (IO3)
- net RXD0: now also TP18.1
- net SCL: now also U8.7 (SCL)
- net SDA: now also R48.1, U8.8 (SDA); no longer U1.12 (IO8)
- net TXD0: now also TP11.1
- net VSYNC: now also R62.2; no longer U1.35 (IO42)
- net ~{RESET}: now also R39.1; no longer U1.3 (EN)
- net at J2.19 (Pin_19), J2.23 (Pin_23): now also R58.2, R65.2; no longer U1.24 (IO47), U1.31 (IO38)
- net at U5.10 (P5): now also TP20.1
- net IO35: now reaches U1.28 (IO35)
- net IO35: now also TP7.1
- net IO36: now reaches U1.29 (IO36)
- net IO36: now also TP8.1
- net IO37: now reaches U1.30 (IO37)
- net IO37: now also TP9.1
- net at U1.4 (IO4): now also R44.2
- net at U5.11 (P6): now also TP14.1
- removed net +5V: C1.1, C10.1, C2.1, C3.1, C4.1, C9.1, D1.2 (A), D2.1 (K), L1.1, R4.1, R5.2, TP1.1, U2.5 (VBUS), U3.1 (VIN), U4.5 (VIN)
- net A0 renamed IO17
- net IO17: now also TP19.1
- net A1 renamed LED_CTRL
- net LED_CTRL: now also R56.1; no longer U1.9 (IO16)
- net CS: no longer names the net of U1.8 (IO15)
- net CS: now also R55.2; no longer R19.1
- net SCK: no longer names the net of U1.5 (IO5)
- net SCK: now also R45.2
- new net: R48.2, U1.12 (IO8)
- new net: R43.2, U1.15 (IO3)
- new net: R64.1, U1.16 (IO46)
- new net: R49.2, U1.17 (IO9)
- new net: R50.2, U1.18 (IO10)
- new net: R51.2, U1.19 (IO11)
- new net: R52.2, U1.20 (IO12)
- new net: R53.2, U1.21 (IO13)
- new net: R54.2, U1.22 (IO14)
- new net: R57.1, U1.23 (IO21)
- new net: R65.1, U1.24 (IO47)
- new net: R66.1, U1.25 (IO48)
- new net: R63.1, U1.26 (IO45)
- new net: R40.2, U1.27 (IO0)
- new net: R39.2, U1.3 (EN)
- new net: R58.1, U1.31 (IO38)
- new net: R59.1, U1.32 (IO39)
- new net: R60.1, U1.33 (IO40)
- new net: R61.1, U1.34 (IO41)
- new net: R62.1, U1.35 (IO42)
- new net: R42.2, U1.38 (IO2)
- new net: R41.2, U1.39 (IO1)
- new net: R46.2, U1.6 (IO6)
- new net: R47.2, U1.7 (IO7)
- new net: R56.2, U1.9 (IO16)
- new net: D5.1 (K), Q1.S, R35.1
- new net: D7.1 (K), J3.2 (Pin_2), R34.1
- new net: TP23.1, U9.9 (DET_B)
- new net: D8.1 (K), R68.1, U9.1 (DAT2)
- new net: R72.1, U9.8 (DAT1)
- new net: R67.2, TP15.1, U8.6 (QSTRT)
- new net: D6.1 (K), R37.1
- new net: R37.2, U7.1 (STAT)
- new net: D14.1 (K), R73.2
- new net: C16.2, R38.2, U7. (Vbat)
- new net: R36.1, U7.5 (PROG)
- new net: TP22.1, U9.10 (DET_A)
- new net +BATT: C18.1, Q1.D, R34.2, R38.1, TP16.1, U8.2 (CELL)
- new net HB_LED: D14.2 (A), R44.1
- new net SD_CS: D9.1 (K), R19.1, R55.1, R69.1, U9.2 (DAT3/CD)
- new net SPI_SCK: D12.1 (K), R45.1, U9.5 (CLK)
- new net VBUS: C1.1, C17.2, C2.1, D1.2 (A), D2.1 (K), D5.2 (A), D6.2 (A), Q1.G, R33.2, R5.2, TP1.1, U2.5 (VBUS), U7.4 (Vdd)
- new net Vin: C3.1, C4.1, R35.2, R4.1, TP17.1, U3.1 (VIN)
- new net ~{BATT_ALRT}: TP21.1, U8.5 (~{ALRT})
Other:
- note added: "MCU/IO"
- note added: "Power Input/Battery"
- note added: "RGB666 Display"
- moved on the sheet: C1, C10, C11, C12, C13, C14, C2, C3, C4, C5, C7, C8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

Commit message: first pass schematic design, open ERC items
Parts:
- removed D10, D11, D12, D13, D8, D9: ESD5Zxx, Diode_SMD:D_SOD-523, symbol Diode:ESD5Zxx
- removed R68, R69, R70, R71, R72: 5.1k, symbol Device:R_Small_US
- removed TP12: TestPoint, symbol Connector:TestPoint
- removed TP18, TP19, TP22, TP23: TestPoint_Alt, symbol Connector:TestPoint_Alt
- removed U9: 5033981892, symbol 5033981892:5033981892
- added C15: 220pF, symbol Device:C_Small
- added C22: 10uF, symbol Device:C_Small
- added C23, C24: 100nF, symbol Device:C_Small
- added D8: SMAJ5.0A, Diode_SMD:D_SMA, symbol Diode:SMAJ5.0A
- added J4: 533980271, symbol Connector_Generic_MountingPin:Conn_01x02_MountingPin
- added L2, L3: L_Ferrite_Small, symbol Device:L_Ferrite_Small
- added R21, R22: DNI, symbol Device:R_Small_US
- added R29: 820, symbol Device:R_Small_US
- added R30, R31: 0, symbol Device:R_Small_US
- added R32: 5.1k, symbol Device:R_Small_US
- added TP10: TestPoint_Alt, symbol Connector:TestPoint_Alt
- added U6: MAX98357A, Package_DFN_QFN:TQFN-16-1EP_3x3mm_P0.5mm_EP1.23x1.23mm, symbol Audio:MAX98357A
- C17: value 100nF -> 10uF
- C19: value 1uF -> 220pF
- J1: value USB_C_Receptacle_USB2.0_14P -> USB4220-03-0880-C
- J2: value Conn_01x40 -> F300-1B7H1-11040-E100
- J3: value JST-PH -> B2B-PH-SM4-TB
- Q1: symbol Device:Q_PMOS -> Transistor_FET:Q_PMOS_DGS
- R67: value 5.1k -> 0
Connections:
- net +3V3: now also C22.1, C23.1, R22.2, R29.2, R30.2, R32.1; no longer C19.1, C6.2, U8.3 (Vdd)
- net +BATT: now also C6.2, Q1.1 (D), U8.3 (Vdd); no longer Q1.D
- net EXP_IRQ: now also R32.2, TP10.1
- net GND: now also C15.2, C22.2, C23.2, C24.2, D8.2 (A2), J4.MP (MountPin), R21.1, U6.11 (GND), U6.15 (GND), U6.17 (PAD), U6.3 (GND)
- net RXD0: now also R31.2, U6.14 (LRCLK); no longer U1.36 (RXD0)
- net VBUS: now also Q1.2 (G), C24.1; no longer Q1.G
- net at D5.1 (K), R35.1: now also Q1.3 (S); no longer Q1.S
- net at D7.1 (K), J3.2 (Pin_2), R34.1: now also D8.1 (A1)
- net at R9.2, TP13.1, U4.4 (CTRL): no longer R11.2
- net IO17: no longer names the net of U1.10 (IO17)
- net IO17: now also R11.1
- net LED_CTRL renamed A1
- net A1: now also U6.1 (DIN); no longer R11.1
- new net: R31.1, U1.36 (RXD0)
- new net: R29.1, U6.4 (~{SD_MODE})
- new net: C19.1, J4.1 (Pin_1), L2.2
- new net: L3.1, U6.10 (OUTN)
- new net: C15.1, J4.2 (Pin_2), L3.2
- new net: R21.2, R22.1, U6.2 (GAIN_SLOT)
- new net: R30.1, U6.7 (VDD), U6.8 (VDD)
- new net: L2.1, U6.9 (OUTP)
- new net A0: R11.2, U6.16 (BCLK)
Other:
- note added: "Audio"
- note added: "HD40015C40"
- note added: "Power"
- note removed: "Power Input/Battery"
- note removed: "RGB666 Display"
- moved on the sheet: C1, C10, C11, C12, C13, C14, C16, C17, C18, C2, C20, C21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

Commit message: clear ERC errors, correct mislabeled nets
Parts:
- removed C3: 100nF, symbol Device:C_Small
- removed L2, L3: L_Ferrite_Small, symbol Device:L_Ferrite_Small
- added R56, R57: 0, symbol Device:R_Small_US
- added TP15, TP16, TP17: TestPoint_Alt, symbol Connector:TestPoint_Alt
- C22: renamed from C15; value 220pF -> DNI
- C23: renamed from C19; value 220pF -> DNI
- L1: value L_Small -> 6.8uH
- R35: renamed from R29; value 820 -> 5.1k
- renumbered C9 to C1, C12 to C10, C16 to C11, C21 to C12, C6 to C13, C4 to C14, C20 to C15, C5 to C16, C14 to C17, C8 to C18, C22 to C19, C10 to C2, C23 to C20, C7 to C21, C17 to C3, C24 to C4, C1 to C5, C18 to C6, C13 to C7, C11 to C8, C2 to C9, D7 to D1, D8 to D2, D2 to D3, D6 to D4, D4 to D5, D1 to D6, D5 to D7, D3 to D8, D14 to D9, J3 to J1, J1 to J2, J2 to J3, R36 to R10, R33 to R11, R16 to R12, R35 to R13, R67 to R14, R12 to R15, R13 to R16, R14 to R17, R15 to R18, R17 to R19, R9 to R2, R4 to R20, R6 to R21, R25 to R22, R27 to R23, R28 to R24, R23 to R25, R7 to R27, R24 to R28, R73 to R29, R5 to R3, R18 to R30, R19 to R31, R8 to R32, R32 to R33, R22 to R34, R21 to R36, R40 to R37, R42 to R38, R44 to R39, R2 to R4, R46 to R40, R48 to R41, R50 to R42, R52 to R43, R54 to R44, R56 to R45, R39 to R46, R41 to R47, R43 to R48, R45 to R49, R34 to R5, R47 to R50, R49 to R51, R51 to R52, R55 to R54, R30 to R55, R11 to R58, R57 to R59, R10 to R6, R58 to R60, R60 to R61, R64 to R63, R66 to R64, R31 to R65, R59 to R66, R61 to R67, R63 to R68, R65 to R69, R37 to R7, R20 to R70, R38 to R8, R3 to R9, TP2 to TP1, TP3 to TP10, TP10 to TP11, TP20 to TP12, TP14 to TP13, TP4 to TP14, TP11 to TP18, TP7 to TP19, TP13 to TP2, TP8 to TP20, TP9 to TP21, TP1 to TP3, TP16 to TP4, TP6 to TP5, TP5 to TP6, TP15 to TP7, TP17 to TP8, TP21 to TP9, U2 to U1, U4 to U2, U7 to U3, U8 to U4, U3 to U5, U5 to U6, U6 to U7, U1 to U8
Connections:
- net PLCK is gone; now on net PCLK: R19.1
- net BACKLIGHT: now also R2.2, TP2.1, U2.4 (CTRL)
- net MISO: now also TP16.1
- net MOSI: now also TP17.1
- net B3: now reaches J3.19 (Pin_19), R60.2
- net B3: no longer J3.23 (Pin_23), R69.2
- net at C23.1, J4.1 (Pin_1): now also R56.2
- net at U7.10 (OUTN): now also R57.1
- net at C22.1, J4.2 (Pin_2): now also R57.2
- net at U7.9 (OUTP): now also R56.1
- net SD_CS renamed CS
- net SPI_SCK renamed SCK
- net SCK: now also TP15.1
- new net G1: J3.23 (Pin_23), R69.2
Other:
- moved on the sheet: C16, C6, D8, D9, R20, R21, R27, R29, R30, R31, R5, R70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

Commit message: add most footprints, some non-generic ones still left
Parts:
- C1, C10, C11, C12, C13, C14, C15, C16, C17, C18, C19, C2, C20, C21, C22, C23, C3, C4, C5, C6, C7, C8, C9: footprint (none) -> Capacitor_SMD:C_0805_2012Metric_Pad1.18x1.45mm_HandSolder
- D4, D6, D8, D9: footprint (none) -> LED_SMD:LED_0805_2012Metric_Pad1.15x1.40mm_HandSolder
- J1: footprint (none) -> B2B-PH-SM4-TBLFSN_JST:B2B-PH-SM4-TB
- J2: footprint (none) -> USB4220-03:USB4220-03
- L1: footprint (none) -> Inductor_SMD:L_0805_2012Metric_Pad1.05x1.20mm_HandSolder
- Q1: footprint (none) -> Package_TO_SOT_SMD:SOT-23; symbol Transistor_FET:Q_PMOS_DGS -> Transistor_FET:Q_PMOS_GSD
- R1, R10, R11, R12, R13, R14, R15, R16, R17, R18, R19, R2, R20, R21, R22, R23, R24, R25, R26, R27, R28, R29, R3, R30, R31, R32, R33, R34, R35, R36, R37, R38, R39, R4, R40, R41, R42, R43, R44, R45, R46, R47, R48, R49, R5, R50, R51, R52, R53, R54, R55, R56, R57, R58, R59, R6, R60, R61, R62, R63, R64, R65, R66, R67, R68, R69, R7, R70, R8, R9: footprint (none) -> Resistor_SMD:R_0805_2012Metric_Pad1.20x1.40mm_HandSolder
- SW1, SW2: footprint (none) -> skrpace010:SKRPACE010
- TP1, TP10, TP14, TP2, TP3, TP4, TP5, TP6, TP8: footprint (none) -> TestPoint:TestPoint_Pad_D2.0mm
- TP11, TP12, TP13, TP15, TP16, TP17, TP18, TP19, TP20, TP21, TP7, TP9: footprint (none) -> TestPoint:TestPoint_THTPad_D2.5mm_Drill1.2mm
- U2: footprint (none) -> Package_TO_SOT_SMD:SOT-353_SC-70-5_Handsoldering
- U3: footprint (none) -> Package_TO_SOT_SMD:SOT-23-5_HandSoldering
- U4: footprint (none) -> Package_DFN_QFN:DFN-8-1EP_2x2mm_P0.5mm_EP0.8x1.6mm
- U6: footprint (none) -> Package_SO:TSSOP-16_4.4x5mm_P0.65mm
Connections:
- net +BATT: now also Q1.3 (D); no longer Q1.1 (D)
- net VBUS: now also Q1.1 (G); no longer Q1.2 (G)
- net at D7.1 (K), R13.1: now also Q1.2 (S); no longer Q1.3 (S)
- net at C11.2, R8.2: now also U3.3 (Vbat); no longer U3. (Vbat)
