File: ecad/dbz-radar/dbz-radar.kicad_pcb (KiCad board)
At the start: 4 copper layers, 125.2 x 122.2 mm, 140 parts, among them J1 B2B-PH-SM4-TB, J2 USB4220-03-0880-C, J3 XF2M-4015-1A, J4 533980271, J5 Conn_01x12_Pin, Q1 Q_PMOS, SW1 SKRPACE010, SW2 SKRPACE010, SW3 1-825027-7, U1 USBLC6-2SC6, U2 TPS61169, U3 MCP738311/2, U4 MAX17048/9, U5 AP2112K-3.3, U6 PCA9554, U7 MAX98357A, U8 ESP32-S3-WROOM-1

Commit message: finalize layout
Parts:
- moved TP1 10.7 mm to (103.3, 100.5)
- moved R32 5.79 mm to (155.8, 36.9), turned to -45 degrees
- moved C19 5.70 mm to (106.6, 48.9), turned to -45 degrees
- moved C20 5.10 mm to (103.7, 48.8), turned to 135 degrees
- moved D1 3.96 mm to (106.9, 98.0)
- moved D2 3.93 mm to (110.3, 97.7)
- moved C18 3.14 mm to (154.4, 38.3), turned to 135 degrees
- moved TP14 2.52 mm to (149.9, 34.1)
- moved R1 2.14 mm to (129.0, 59.4)
- moved D3 1.55 mm to (119.6, 68.8), turned to 90 degrees
- moved C5 1.48 mm to (116.7, 69.8)
- moved C9 1.48 mm to (115.2, 71.4)
- moved R11 1.48 mm to (111.9, 74.5)
- moved R9 1.48 mm to (109.9, 69.3)
- moved D6 1.48 mm to (113.5, 72.9)
Connections:
- J2 pad A6: /USB_CONN_D+ -> /USB_D+
- J2 pad A7: /USB_CONN_D- -> /USB_D-
- J2 pad B6: /USB_CONN_D+ -> /USB_D+
- J2 pad B7: /USB_CONN_D- -> /USB_D-
- J5 pad 13: unconnected-(J5-Pin_13-Pad13) -> +3V3
- U1 pad 1: /USB_CONN_D+ -> /USB_D+
- U1 pad 3: /USB_CONN_D- -> /USB_D-
Routing:
- net /USB_D+: track 42.3 -> 58.3 mm, vias 2 -> 4
- net /USB_D-: track 42.3 -> 58.2 mm, vias 2 -> 4
- net /USB_CONN_D+: track 13.3 -> 0.00 mm, vias 2 -> 0
- net /USB_CONN_D-: track 11.8 -> 0.00 mm, vias 2 -> 0
- net /~{RESET}: track 30.6 -> 36.1 mm
- net +3V3: track 45.8 -> 50.8 mm, vias 33 -> 32
- net /MOSI: track 76.7 -> 75.4 mm
- net GND: track 11.3 -> 12.4 mm, vias 73 -> 173
- net Net-(J2-CC1): track 6.69 -> 7.77 mm
- net /SCL: track 210.0 -> 210.9 mm
- net /MISO: track 73.7 -> 72.9 mm
- net /DE: track 89.7 -> 90.5 mm
- net /PCLK: track 81.2 -> 81.9 mm
- net Net-(U8-IO18): track 29.1 -> 29.8 mm
- net /SCK: track 71.0 -> 70.3 mm
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
Commit message: add all 3D shapes, add helpful text so silkscreen
Parts:
- removed D2: SMAJ5.0A, Diode_SMD:D_SMA
Connections:
- net /EXP_IRQ renamed /~{EXP_IRQ}
Routing:
- net /TP_IRQ: track 79.5 -> 78.9 mm
- net GND: vias 173 -> 177
Other:
- board text added: "24V"
- board text added: "3V3"
- board text added: "A0"
- board text added: "A1"
- board text added: "B1"
- board text added: "B2"
- board text added: "B3"
- board text added: "B4"
- board text added: "B5"
- board text added: "BACKLIGHT"
- board text added: "BATT"
- board text added: "BATT_MON_ALRT"
- board text added: "BOOT"
- board text added: "BUTTON"
- board text added: "CS"
- board text added: "DE"
- board text added: "Dragon Ball Radar v0.1.0 extralongdivision.com"
- board text added: "G0"
- board text added: "G1"
- board text added: "G2"
- board text added: "G3"
- board text added: "G4"
- board text added: "G5"
- board text added: "GND"
- board text added: "HSYNC"
- board text added: "I2C_P6"
- board text added: "IO35"
- board text added: "IO36"
- board text added: "IO37"
- board text added: "LEDK"
- board text added: "MISO"
- board text added: "MOSI"
- board text added: "PCLK"
- board text added: "R1"
- board text added: "R2"
- board text added: "R3"
- board text added: "R4"
- board text added: "R5"
- board text added: "RESET"
- board text added: "RST"
- board text added: "RX0"
- board text added: "SCK"
- board text added: "SCL"
- board text added: "SDA"
- board text added: "TX0"
- board text added: "VBUS"
- board text added: "VSYNC"
- board text added: "Vin"
- board text added: "~{BATT_ALRT}"
- board text added: "~{EXP_IRQ}"
- board text added: "~{RESET}"

Commit message: move MCU to fit in MCAD
Parts:
- moved SW2 11.4 mm to (161.6, 92.5)
- moved R48 8.14 mm to (149.2, 64.7)
- moved R69 8.14 mm to (163.7, 79.2)
- moved R51 8.14 mm to (152.3, 67.8)
- moved R63 8.14 mm to (150.8, 66.3)
- moved R37 8.14 mm to (168.6, 84.1)
- moved R42 8.14 mm to (153.9, 69.5)
- moved R43 8.14 mm to (157.2, 72.7)
- moved R44 8.14 mm to (160.4, 76.0)
- moved R52 8.14 mm to (155.6, 71.1)
- moved R53 8.14 mm to (158.8, 74.4)
- moved R59 8.14 mm to (162.1, 77.6)
- moved R64 8.14 mm to (165.3, 80.9)
- moved R68 8.14 mm to (167.0, 82.4)
- moved U8 7.08 mm to (171.2, 61.0)
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Routing:
- net /USB_D+: track 58.3 -> 49.9 mm
- net /USB_D-: track 58.2 -> 49.8 mm
- net /R5: track 80.0 -> 72.2 mm
- net /R2: track 76.6 -> 68.8 mm
- net /R4: track 78.9 -> 71.1 mm
- net /G5: track 74.1 -> 66.3 mm
- net /G3: track 71.7 -> 64.0 mm
- net /G1: track 69.4 -> 61.7 mm
- net /R3: track 77.7 -> 70.0 mm
- net /G2: track 70.6 -> 62.8 mm
- net /G4: track 72.9 -> 65.1 mm
- net /R1: track 76.7 -> 69.0 mm
- net /BOOT0_B4: track 65.9 -> 58.2 mm
- net /G0: track 68.3 -> 60.5 mm
- net /B5: track 67.1 -> 59.5 mm
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